File: keypad-kicad-proj/keypad/button-led-strip.kicad_sch (KiCad schematic)
At the start: 13 parts, among them U10 SK6812MINI-E, U11 SK6812MINI-E, U12 SK6812MINI-E, U13 SK6812MINI-E, U14 SK6812MINI-E, U3 SK6812MINI-E, U4 SK6812MINI-E, U5 SK6812MINI-E, U6 SK6812MINI-E, U7 SK6812MINI-E, U8 SK6812MINI-E, U9 SK6812MINI-E

Commit message: rest of the schematic
Other:
- title: (none) -> Keypad board
Changed lines of the file:
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@@
 (kicad_sch (version 20230121) (generator eeschema)
   (paper "A4")
+  (title_block
+    (title "Keypad board")
+    (date "2023-11-15")
+    (rev "1.1")
+  )
   (junction (at 113.03 72.39) (diameter 0) (color 0 0 0 0)
   )
@@
           (reference "#PWR016") (unit 1)
         )
-        (path "/26078c39-1d91-4154-8719-da74cb453e74/98588952-669a-4c5f-948d-9729b3b04ace"
-          (reference "#PWR030") (unit 1)
+        (path "/26078c39-1d91-4154-8719-da74cb453e74/3159a0fd-9cfb-4836-b001-4197fb47d6b2/18d73d02-d240-4308-a5a7-c3da203c7f9c"
+          (reference "#PWR058") (unit 1)
         )
       )
@@
           (reference "U4") (unit 1)
         )
-        (path "/26078c39-1d91-4154-8719-da74cb453e74/98588952-669a-4c5f-948d-9729b3b04ace"
-          (reference "U16") (unit 1)
+        (path "/26078c39-1d91-4154-8719-da74cb453e74/3159a0fd-9cfb-4836-b001-4197fb47d6b2/18d73d02-d240-4308-a5a7-c3da203c7f9c"
+          (reference "U5") (unit 1)
         )
       )
@@
           (reference "U6") (unit 1)
         )
-        (path "/26078c39-1d91-4154-8719-da74cb453e74/98588952-669a-4c5f-948d-9729b3b04ace"
-          (reference "U18") (unit 1)
+        (path "/26078c39-1d91-4154-8719-da74cb453e74/3159a0fd-9cfb-4836-b001-4197fb47d6b2/18d73d02-d240-4308-a5a7-c3da203c7f9c"
+          (reference "U7") (unit 1)
         )
       )
@@
           (reference "U3") (unit 1)
         )
-        (path "/26078c39-1d91-4154-8719-da74cb453e74/98588952-669a-4c5f-948d-9729b3b04ace"
-          (reference "U15") (unit 1)
+        (path "/26078c39-1d91-4154-8719-da74cb453e74/3159a0fd-9cfb-4836-b001-4197fb47d6b2/18d73d02-d240-4308-a5a7-c3da203c7f9c"
+          (reference "U4") (unit 1)
         )
       )
@@
           (reference "#PWR020") (unit 1)
         )
-        (path "/26078c39-1d91-4154-8719-da74cb453e74/98588952-669a-4c5f-948d-9729b3b04ace"
-          (reference "#PWR034") (unit 1)
+        (path "/26078c39-1d91-4154-8719-da74cb453e74/3159a0fd-9cfb-4836-b001-4197fb47d6b2/18d73d02-d240-4308-a5a7-c3da203c7f9c"
+          (reference "#PWR062") (unit 1)
         )
       )
@@
           (reference "R5") (unit 1)
         )
-        (path "/26078c39-1d91-4154-8719-da74cb453e74/98588952-669a-4c5f-948d-9729b3b04ace"
-          (reference "R6") (unit 1)
+        (path "/26078c39-1d91-4154-8719-da74cb453e74/3159a0fd-9cfb-4836-b001-4197fb47d6b2/18d73d02-d240-4308-a5a7-c3da203c7f9c"
+          (reference "R20") (unit 1)
         )
       )
@@
           (reference "#PWR027") (unit 1)
         )
-        (path "/26078c39-1d91-4154-8719-da74cb453e74/98588952-669a-4c5f-948d-9729b3b04ace"
-          (reference "#PWR028") (unit 1)
+        (path "/26078c39-1d91-4154-8719-da74cb453e74/3159a0fd-9cfb-4836-b001-4197fb47d6b2/18d73d02-d240-4308-a5a7-c3da203c7f9c"
+          (reference "#PWR056") (unit 1)
         )
       )
@@
           (reference "U5") (unit 1)
         )
-        (path "/26078c39-1d91-4154-8719-da74cb453e74/98588952-669a-4c5f-948d-9729b3b04ace"
-          (reference "U17") (unit 1)
+        (path "/26078c39-1d91-4154-8719-da74cb453e74/3159a0fd-9cfb-4836-b001-4197fb47d6b2/18d73d02-d240-4308-a5a7-c3da203c7f9c"
+          (reference "U6") (unit 1)
         )
       )
@@
           (reference "U10") (unit 1)
         )
-        (path "/26078c39-1d91-4154-8719-da74cb453e74/98588952-669a-4c5f-948d-9729b3b04ace"
-          (reference "U22") (unit 1)
+        (path "/26078c39-1d91-4154-8719-da74cb453e74/3159a0fd-9cfb-4836-b001-4197fb47d6b2/18d73d02-d240-4308-a5a7-c3da203c7f9c"
+          (reference "U11") (unit 1)
         )
       )
@@
           (reference "U13") (unit 1)
         )
-        (path "/26078c39-1d91-4154-8719-da74cb453e74/98588952-669a-4c5f-948d-9729b3b04ace"
-          (reference "U25") (unit 1)
+        (path "/26078c39-1d91-4154-8719-da74cb453e74/3159a0fd-9cfb-4836-b001-4197fb47d6b2/18d73d02-d240-4308-a5a7-c3da203c7f9c"
+          (reference "U14") (unit 1)
         )
       )
@@
           (reference "U14") (unit 1)
         )
-        (path "/26078c39-1d91-4154-8719-da74cb453e74/98588952-669a-4c5f-948d-9729b3b04ace"
-          (reference "U26") (unit 1)
+        (path "/26078c39-1d91-4154-8719-da74cb453e74/3159a0fd-9cfb-4836-b001-4197fb47d6b2/18d73d02-d240-4308-a5a7-c3da203c7f9c"
+          (reference "U27") (unit 1)
         )
       )
@@
           (reference "U7") (unit 1)
         )
-        (path "/26078c39-1d91-4154-8719-da74cb453e74/98588952-669a-4c5f-948d-9729b3b04ace"
-          (reference "U19") (unit 1)
+        (path "/26078c39-1d91-4154-8719-da74cb453e74/3159a0fd-9cfb-4836-b001-4197fb47d6b2/18d73d02-d240-4308-a5a7-c3da203c7f9c"
+          (reference "U8") (unit 1)
         )
       )
@@
           (reference "U11") (unit 1)
         )
-        (path "/26078c39-1d91-4154-8719-da74cb453e74/98588952-669a-4c5f-948d-9729b3b04ace"
-          (reference "U23") (unit 1)
+        (path "/26078c39-1d91-4154-8719-da74cb453e74/3159a0fd-9cfb-4836-b001-4197fb47d6b2/18d73d02-d240-4308-a5a7-c3da203c7f9c"
+          (reference "U12") (unit 1)
         )
       )
@@
           (reference "U12") (unit 1)
         )
-        (path "/26078c39-1d91-4154-8719-da74cb453e74/98588952-669a-4c5f-948d-9729b3b04ace"
-          (reference "U24") (unit 1)
+        (path "/26078c39-1d91-4154-8719-da74cb453e74/3159a0fd-9cfb-4836-b001-4197fb47d6b2/18d73d02-d240-4308-a5a7-c3da203c7f9c"
+          (reference "U13") (unit 1)
         )
       )
@@
           (reference "U9") (unit 1)
         )
-        (path "/26078c39-1d91-4154-8719-da74cb453e74/98588952-669a-4c5f-948d-9729b3b04ace"
-          (reference "U21") (unit 1)
+        (path "/26078c39-1d91-4154-8719-da74cb453e74/3159a0fd-9cfb-4836-b001-4197fb47d6b2/18d73d02-d240-4308-a5a7-c3da203c7f9c"
+          (reference "U10") (unit 1)
         )
       )
@@
           (reference "U8") (unit 1)
         )
-        (path "/26078c39-1d91-4154-8719-da74cb453e74/98588952-669a-4c5f-948d-9729b3b04ace"
-          (reference "U20") (unit 1)
+        (path "/26078c39-1d91-4154-8719-da74cb453e74/3159a0fd-9cfb-4836-b001-4197fb47d6b2/18d73d02-d240-4308-a5a7-c3da203c7f9c"
+          (reference "U9") (unit 1)
         )
       )
@@
           (reference "#PWR017") (unit 1)
         )
-        (path "/26078c39-1d91-4154-8719-da74cb453e74/98588952-669a-4c5f-948d-9729b3b04ace"
-          (reference "#PWR031") (unit 1)
+        (path "/26078c39-1d91-4154-8719-da74cb453e74/3159a0fd-9cfb-4836-b001-4197fb47d6b2/18d73d02-d240-4308-a5a7-c3da203c7f9c"
+          (reference "#PWR059") (unit 1)
         )
       )
@@
           (reference "#PWR023") (unit 1)
         )
-        (path "/26078c39-1d91-4154-8719-da74cb453e74/98588952-669a-4c5f-948d-9729b3b04ace"
-          (reference "#PWR037") (unit 1)
+        (path "/26078c39-1d91-4154-8719-da74cb453e74/3159a0fd-9cfb-4836-b001-4197fb47d6b2/18d73d02-d240-4308-a5a7-c3da203c7f9c"
+          (reference "#PWR065") (unit 1)
         )
       )
@@
           (reference "#PWR018") (unit 1)
         )
-        (path "/26078c39-1d91-4154-8719-da74cb453e74/98588952-669a-4c5f-948d-9729b3b04ace"
-          (reference "#PWR032") (unit 1)
+        (path "/26078c39-1d91-4154-8719-da74cb453e74/3159a0fd-9cfb-4836-b001-4197fb47d6b2/18d73d02-d240-4308-a5a7-c3da203c7f9c"
+          (reference "#PWR060") (unit 1)
         )
       )
@@
           (reference "#PWR025") (unit 1)
         )
-        (path "/26078c39-1d91-4154-8719-da74cb453e74/98588952-669a-4c5f-948d-9729b3b04ace"
-          (reference "#PWR039") (unit 1)
+        (path "/26078c39-1d91-4154-8719-da74cb453e74/3159a0fd-9cfb-4836-b001-4197fb47d6b2/18d73d02-d240-4308-a5a7-c3da203c7f9c"
+          (reference "#PWR067") (unit 1)
         )
       )
@@
           (reference "#PWR026") (unit 1)
         )
-        (path "/26078c39-1d91-4154-8719-da74cb453e74/98588952-669a-4c5f-948d-9729b3b04ace"
-          (reference "#PWR040") (unit 1)
+        (path "/26078c39-1d91-4154-8719-da74cb453e74/3159a0fd-9cfb-4836-b001-4197fb47d6b2/18d73d02-d240-4308-a5a7-c3da203c7f9c"
+          (reference "#PWR068") (unit 1)
         )
       )
@@
           (reference "#PWR022") (unit 1)
         )
-        (path "/26078c39-1d91-4154-8719-da74cb453e74/98588952-669a-4c5f-948d-9729b3b04ace"
-          (reference "#PWR036") (unit 1)
+        (path "/26078c39-1d91-4154-8719-da74cb453e74/3159a0fd-9cfb-4836-b001-4197fb47d6b2/18d73d02-d240-4308-a5a7-c3da203c7f9c"
+          (reference "#PWR064") (unit 1)
         )
       )
@@
           (reference "#PWR021") (unit 1)
         )
-        (path "/26078c39-1d91-4154-8719-da74cb453e74/98588952-669a-4c5f-948d-9729b3b04ace"
-          (reference "#PWR035") (unit 1)
+        (path "/26078c39-1d91-4154-8719-da74cb453e74/3159a0fd-9cfb-4836-b001-4197fb47d6b2/18d73d02-d240-4308-a5a7-c3da203c7f9c"
+          (reference "#PWR063") (unit 1)
         )
       )
@@
           (reference "#PWR019") (unit 1)
         )
-        (path "/26078c39-1d91-4154-8719-da74cb453e74/98588952-669a-4c5f-948d-9729b3b04ace"
-          (reference "#PWR033") (unit 1)
+        (path "/26078c39-1d91-4154-8719-da74cb453e74/3159a0fd-9cfb-4836-b001-4197fb47d6b2/18d73d02-d240-4308-a5a7-c3da203c7f9c"
+          (reference "#PWR061") (unit 1)
         )
       )
@@
           (reference "#PWR015") (unit 1)
         )
-        (path "/26078c39-1d91-4154-8719-da74cb453e74/98588952-669a-4c5f-948d-9729b3b04ace"
-          (reference "#PWR029") (unit 1)
+        (path "/26078c39-1d91-4154-8719-da74cb453e74/3159a0fd-9cfb-4836-b001-4197fb47d6b2/18d73d02-d240-4308-a5a7-c3da203c7f9c"
+          (reference "#PWR057") (unit 1)
         )
       )
@@
           (reference "#PWR024") (unit 1)
         )
-        (path "/26078c39-1d91-4154-8719-da74cb453e74/98588952-669a-4c5f-948d-9729b3b04ace"
-          (reference "#PWR038") (unit 1)
-        )
-      )
+        (path "/26078c39-1d91-4154-8719-da74cb453e74/3159a0fd-9cfb-4836-b001-4197fb47d6b2/18d73d02-d240-4308-a5a7-c3da203c7f9c"
+          (reference "#PWR066") (unit 1)
+        )
+      )

Commit message: footprints
Parts:
- R5: footprint (none) -> Resistor_SMD:R_0603_1608Metric
- U10, U11, U12, U13, U14, U3, U4, U5, U6, U7, U8, U9: footprint (none) -> PUT_RocketLab_other:SK6812MINI-E
Changed lines of the file:
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@@
       (effects (font (size 1.27 1.27)))
     )
-    (property "Footprint" "" (at 78.74 80.01 0)
+    (property "Footprint" "PUT_RocketLab_other:SK6812MINI-E" (at 78.74 80.01 0)
       (effects (font (size 1.27 1.27)) hide)
     )
@@
       (effects (font (size 1.27 1.27)))
     )
-    (property "Footprint" "" (at 114.3 80.01 0)
+    (property "Footprint" "PUT_RocketLab_other:SK6812MINI-E" (at 114.3 80.01 0)
       (effects (font (size 1.27 1.27)) hide)
     )
@@
       (effects (font (size 1.27 1.27)))
     )
-    (property "Footprint" "" (at 60.96 80.01 0)
+    (property "Footprint" "PUT_RocketLab_other:SK6812MINI-E" (at 60.96 80.01 0)
       (effects (font (size 1.27 1.27)) hide)
     )
@@
       (effects (font (size 1.27 1.27)))
     )
-    (property "Footprint" "" (at 46.99 81.28 0)
+    (property "Footprint" "Resistor_SMD:R_0603_1608Metric" (at 46.99 81.28 0)
       (effects (font (size 1.27 1.27)) hide)
     )
@@
       (effects (font (size 1.27 1.27)))
     )
-    (property "Footprint" "" (at 96.52 80.01 0)
+    (property "Footprint" "PUT_RocketLab_other:SK6812MINI-E" (at 96.52 80.01 0)
       (effects (font (size 1.27 1.27)) hide)
     )
@@
       (effects (font (size 1.27 1.27)))
     )
-    (property "Footprint" "" (at 185.42 80.01 0)
+    (property "Footprint" "PUT_RocketLab_other:SK6812MINI-E" (at 185.42 80.01 0)
       (effects (font (size 1.27 1.27)) hide)
     )
@@
       (effects (font (size 1.27 1.27)))
     )
-    (property "Footprint" "" (at 238.76 80.01 0)
+    (property "Footprint" "PUT_RocketLab_other:SK6812MINI-E" (at 238.76 80.01 0)
       (effects (font (size 1.27 1.27)) hide)
     )
@@
       (effects (font (size 1.27 1.27)))
     )
-    (property "Footprint" "" (at 256.54 80.01 0)
+    (property "Footprint" "PUT_RocketLab_other:SK6812MINI-E" (at 256.54 80.01 0)
       (effects (font (size 1.27 1.27)) hide)
     )
@@
       (effects (font (size 1.27 1.27)))
     )
-    (property "Footprint" "" (at 132.08 80.01 0)
+    (property "Footprint" "PUT_RocketLab_other:SK6812MINI-E" (at 132.08 80.01 0)
       (effects (font (size 1.27 1.27)) hide)
     )
@@
       (effects (font (size 1.27 1.27)))
     )
-    (property "Footprint" "" (at 203.2 80.01 0)
+    (property "Footprint" "PUT_RocketLab_other:SK6812MINI-E" (at 203.2 80.01 0)
       (effects (font (size 1.27 1.27)) hide)
     )
@@
       (effects (font (size 1.27 1.27)))
     )
-    (property "Footprint" "" (at 220.98 80.01 0)
+    (property "Footprint" "PUT_RocketLab_other:SK6812MINI-E" (at 220.98 80.01 0)
       (effects (font (size 1.27 1.27)) hide)
     )
@@
       (effects (font (size 1.27 1.27)))
     )
-    (property "Footprint" "" (at 167.64 80.01 0)
+    (property "Footprint" "PUT_RocketLab_other:SK6812MINI-E" (at 167.64 80.01 0)
       (effects (font (size 1.27 1.27)) hide)
     )
@@
       (effects (font (size 1.27 1.27)))
     )
-    (property "Footprint" "" (at 149.86 80.01 0)
-      (effects (font (size 1.27 1.27)) hide)
-    )
+    (property "Footprint" "PUT_RocketLab_other:SK6812MINI-E" (at 149.86 80.01 0)
+      (effects (font (size 1.27 1.27)) hide)
+    )
