File: keypad-kicad-proj/keypad/micro-sd-connector.kicad_sch (KiCad schematic)
At the start: 8 parts, among them J4 Micro_SD_Card_Det_Hirose_DM3AT

Commit message: footprints
Parts:
- C10: footprint (none) -> Capacitor_SMD:C_0402_1005Metric
- R13, R14, R15: footprint (none) -> Resistor_SMD:R_0603_1608Metric
Changed lines of the file:
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@@
       (effects (font (size 1.27 1.27)) (justify left))
     )
-    (property "Footprint" "" (at 129.54 71.12 0)
+    (property "Footprint" "Resistor_SMD:R_0603_1608Metric" (at 129.54 71.12 0)
       (effects (font (size 1.27 1.27)) hide)
     )
@@
       (effects (font (size 1.27 1.27)) (justify left))
     )
-    (property "Footprint" "" (at 116.84 71.12 0)
+    (property "Footprint" "Resistor_SMD:R_0603_1608Metric" (at 116.84 71.12 0)
       (effects (font (size 1.27 1.27)) hide)
     )
@@
       (effects (font (size 1.27 1.27)) (justify left))
     )
-    (property "Footprint" "" (at 135.89 100.33 0)
+    (property "Footprint" "Capacitor_SMD:C_0402_1005Metric" (at 135.89 100.33 0)
       (effects (font (size 1.27 1.27)) hide)
     )
@@
       (effects (font (size 1.27 1.27)) (justify left))
     )
-    (property "Footprint" "" (at 123.19 71.12 0)
+    (property "Footprint" "Resistor_SMD:R_0603_1608Metric" (at 123.19 71.12 0)
       (effects (font (size 1.27 1.27)) hide)
     )

Commit message: add all footprints & move libs to project specific
Parts:
- J4: footprint (none) -> Connector_Card:microSD_HC_Hirose_DM3D-SF
Changed lines of the file:
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@@
       (effects (font (size 1.27 1.27)))
     )
-    (property "Footprint" "" (at 218.44 67.31 0)
+    (property "Footprint" "Connector_Card:microSD_HC_Hirose_DM3D-SF" (at 218.44 67.31 0)
       (effects (font (size 1.27 1.27)) hide)
     )

Commit message: main layout
Parts:
- C10: footprint Capacitor_SMD:C_0402_1005Metric -> Capacitor_SMD:C_0603_1608Metric
Changed lines of the file:
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@@
       (effects (font (size 1.27 1.27)) (justify left))
     )
-    (property "Footprint" "Capacitor_SMD:C_0402_1005Metric" (at 135.89 100.33 0)
+    (property "Footprint" "Capacitor_SMD:C_0603_1608Metric" (at 135.89 100.33 0)
       (effects (font (size 1.27 1.27)) hide)
     )
