File: keypad-kicad-proj/keypad/io.kicad_sch (KiCad schematic)
At the start: 20 parts, among them SW1 RotaryEncoder, SW2 RotaryEncoder, SW25 SW_SPST

Commit message: footprints
Parts:
- 1: footprint (none) -> PUT_RocketLab_other:CMI9605IC0580T
- C9: footprint (none) -> Capacitor_SMD:C_0603_1608Metric
- D1, D26, D27: footprint (none) -> LED_SMD:LED_0805_2012Metric_Pad1.15x1.40mm_HandSolder
- R16: footprint (none) -> Resistor_SMD:R_0402_1005Metric
- R16: footprint (none) -> Resistor_SMD:R_1210_3225Metric
- R17: footprint (none) -> Resistor_SMD:R_2512_6332Metric
- R18, RV1: footprint (none) -> Resistor_SMD:R_0603_1608Metric
- R19: footprint (none) -> Resistor_SMD:R_0201_0603Metric
- SW25: footprint (none) -> Button_Switch_THT:SW_PUSH-12mm_Wuerth-430476085716
Changed lines of the file:
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@@
       (effects (font (size 1.27 1.27)) (justify left))
     )
-    (property "Footprint" "" (at 64.77 127 0)
+    (property "Footprint" "Capacitor_SMD:C_0603_1608Metric" (at 64.77 127 0)
       (effects (font (size 1.27 1.27)) hide)
     )
@@
       (effects (font (size 1.27 1.27)) (justify right))
     )
-    (property "Footprint" "" (at 53.34 52.07 0)
+    (property "Footprint" "LED_SMD:LED_0805_2012Metric_Pad1.15x1.40mm_HandSolder" (at 53.34 52.07 0)
       (effects (font (size 1.27 1.27)) hide)
     )
@@
       (effects (font (size 1.27 1.27)) (justify left))
     )
-    (property "Footprint" "" (at 156.21 46.99 0)
+    (property "Footprint" "Capacitor_SMD:C_0603_1608Metric" (at 156.21 46.99 0)
       (effects (font (size 1.27 1.27)) hide)
     )
@@
       (effects (font (size 1.27 1.27)) (justify left))
     )
-    (property "Footprint" "" (at 129.54 109.22 0)
+    (property "Footprint" "Capacitor_SMD:C_0603_1608Metric" (at 129.54 109.22 0)
       (effects (font (size 1.27 1.27)) hide)
     )
@@
       (effects (font (size 1.27 1.27)) (justify left))
     )
-    (property "Footprint" "" (at 66.04 60.96 0)
+    (property "Footprint" "Resistor_SMD:R_0603_1608Metric" (at 66.04 60.96 0)
       (effects (font (size 1.27 1.27)) hide)
     )
@@
       (effects (font (size 1.27 1.27)) (justify left))
     )
-    (property "Footprint" "" (at 53.34 60.96 0)
+    (property "Footprint" "Resistor_SMD:R_0201_0603Metric" (at 53.34 60.96 0)
       (effects (font (size 1.27 1.27)) hide)
     )
@@
       (effects (font (size 1.27 1.27)) (justify right))
     )
-    (property "Footprint" "" (at 77.47 52.07 0)
+    (property "Footprint" "LED_SMD:LED_0805_2012Metric_Pad1.15x1.40mm_HandSolder" (at 77.47 52.07 0)
       (effects (font (size 1.27 1.27)) hide)
     )
@@
       (effects (font (size 1.27 1.27)) (justify left))
     )
-    (property "Footprint" "" (at 90.17 52.07 0)
+    (property "Footprint" "PUT_RocketLab_other:CMI9605IC0580T" (at 90.17 52.07 0)
       (effects (font (size 1.27 1.27)) hide)
     )
@@
         )
         (path "/26078c39-1d91-4154-8719-da74cb453e74/3159a0fd-9cfb-4836-b001-4197fb47d6b2"
-          (reference "11?") (unit 1)
+          (reference "B1") (unit 1)
         )
       )
@@
       (effects (font (size 1.27 1.27)) (justify left))
     )
-    (property "Footprint" "" (at 64.77 109.22 0)
+    (property "Footprint" "Capacitor_SMD:C_0603_1608Metric" (at 64.77 109.22 0)
       (effects (font (size 1.27 1.27)) hide)
     )
@@
       (effects (font (size 1.27 1.27)) (justify left))
     )
-    (property "Footprint" "" (at 88.9 60.96 0)
+    (property "Footprint" "Resistor_SMD:R_0402_1005Metric" (at 88.9 60.96 0)
       (effects (font (size 1.27 1.27)) hide)
     )
@@
       (effects (font (size 1.27 1.27)) (justify left))
     )
-    (property "Footprint" "" (at 77.47 60.96 0)
+    (property "Footprint" "Resistor_SMD:R_2512_6332Metric" (at 77.47 60.96 0)
       (effects (font (size 1.27 1.27)) hide)
     )
@@
       (effects (font (size 1.27 1.27)) (justify left))
     )
-    (property "Footprint" "" (at 212.09 109.22 0)
+    (property "Footprint" "Resistor_SMD:R_1210_3225Metric" (at 212.09 109.22 0)
       (effects (font (size 1.27 1.27)) hide)
     )
@@
       (effects (font (size 1.27 1.27)))
     )
-    (property "Footprint" "" (at 148.59 41.91 0)
+    (property "Footprint" "Button_Switch_THT:SW_PUSH-12mm_Wuerth-430476085716" (at 148.59 41.91 0)
       (effects (font (size 1.27 1.27)) hide)
     )
@@
       (effects (font (size 1.27 1.27)) (justify left))
     )
-    (property "Footprint" "" (at 129.54 127 0)
+    (property "Footprint" "Capacitor_SMD:C_0603_1608Metric" (at 129.54 127 0)
       (effects (font (size 1.27 1.27)) hide)
     )
@@
       (effects (font (size 1.27 1.27)) (justify right))
     )
-    (property "Footprint" "" (at 218.44 45.72 0)
+    (property "Footprint" "Resistor_SMD:R_0603_1608Metric" (at 218.44 45.72 0)
       (effects (font (size 1.27 1.27)) hide)
     )
@@
       (effects (font (size 1.27 1.27)) (justify left))
     )
-    (property "Footprint" "" (at 207.01 109.22 0)
+    (property "Footprint" "Resistor_SMD:R_1210_3225Metric" (at 207.01 109.22 0)
       (effects (font (size 1.27 1.27)) hide)
     )
@@
       (effects (font (size 1.27 1.27)) (justify right))
     )
-    (property "Footprint" "" (at 66.04 52.07 0)
-      (effects (font (size 1.27 1.27)) hide)
-    )
+    (property "Footprint" "LED_SMD:LED_0805_2012Metric_Pad1.15x1.40mm_HandSolder" (at 66.04 52.07 0)
+      (effects (font (size 1.27 1.27)) hide)
+    )

Commit message: add all footprints & move libs to project specific
Parts:
- Brd1: footprint (none) -> Connector_PinHeader_1.00mm:PinHeader_1x04_P1.00mm_Vertical
- RV1: footprint Resistor_SMD:R_0603_1608Metric -> PUT_RocketLab_other:PTA30432010CIB102
- SW1, SW2: footprint (none) -> Rotary_Encoder:RotaryEncoder_Alps_EC12E-Switch_Vertical_H20mm
Changed lines of the file:
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@@
       (effects (font (size 1.27 1.27)))
     )
-    (property "Footprint" "" (at 231.14 113.03 0)
+    (property "Footprint" "Connector_PinHeader_1.00mm:PinHeader_1x04_P1.00mm_Vertical" (at 231.14 113.03 0)
       (effects (font (size 1.27 1.27)) hide)
     )
@@
       (effects (font (size 1.27 1.27)) (justify left))
     )
-    (property "Footprint" "" (at 71.12 114.046 0)
+    (property "Footprint" "Rotary_Encoder:RotaryEncoder_Alps_EC12E-Switch_Vertical_H20mm" (at 71.12 114.046 0)
       (effects (font (size 1.27 1.27)) hide)
     )
@@
       (effects (font (size 1.27 1.27)) (justify right))
     )
-    (property "Footprint" "Resistor_SMD:R_0603_1608Metric" (at 218.44 45.72 0)
+    (property "Footprint" "PUT_RocketLab_other:PTA30432010CIB102" (at 218.44 45.72 0)
       (effects (font (size 1.27 1.27)) hide)
     )
@@
       (effects (font (size 1.27 1.27)) (justify left))
     )
-    (property "Footprint" "" (at 134.62 114.046 0)
-      (effects (font (size 1.27 1.27)) hide)
-    )
+    (property "Footprint" "Rotary_Encoder:RotaryEncoder_Alps_EC12E-Switch_Vertical_H20mm" (at 134.62 114.046 0)
+      (effects (font (size 1.27 1.27)) hide)
+    )

Commit message: inital pcb layout
Parts:
- SW25: value SW_SPST -> SW_RST; footprint Button_Switch_THT:SW_PUSH-12mm_Wuerth-430476085716 -> Button_Switch_THT:SW_PUSH_6mm
Changed lines of the file:
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@@
       (effects (font (size 1.27 1.27)))
     )
-    (property "Value" "SW_SPST" (at 148.59 38.1 0)
+    (property "Value" "SW_RST" (at 148.59 38.1 0)
       (effects (font (size 1.27 1.27)))
     )
-    (property "Footprint" "Button_Switch_THT:SW_PUSH-12mm_Wuerth-430476085716" (at 148.59 41.91 0)
+    (property "Footprint" "Button_Switch_THT:SW_PUSH_6mm" (at 148.59 41.91 0)
       (effects (font (size 1.27 1.27)) hide)
     )

Commit message: pcb layout update
Parts:
- Brd1: footprint Connector_PinHeader_1.00mm:PinHeader_1x04_P1.00mm_Vertical -> PUT_RocketLab_other:128x64OLED_V2
Changed lines of the file:
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@@
       (effects (font (size 1.27 1.27)))
     )
-    (property "Footprint" "Connector_PinHeader_1.00mm:PinHeader_1x04_P1.00mm_Vertical" (at 231.14 113.03 0)
+    (property "Footprint" "PUT_RocketLab_other:128x64OLED_V2" (at 231.14 113.03 0)
       (effects (font (size 1.27 1.27)) hide)
     )

Commit message: main layout
Parts:
- R16: footprint Resistor_SMD:R_0402_1005Metric -> Resistor_SMD:R_0603_1608Metric
- R16: footprint Resistor_SMD:R_1210_3225Metric -> Resistor_SMD:R_0603_1608Metric
- R17: footprint Resistor_SMD:R_2512_6332Metric -> Resistor_SMD:R_0805_2012Metric
- R19: footprint Resistor_SMD:R_0201_0603Metric -> Resistor_SMD:R_0603_1608Metric
Changed lines of the file:
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@@
       (effects (font (size 1.27 1.27)) (justify left))
     )
-    (property "Footprint" "Resistor_SMD:R_0201_0603Metric" (at 53.34 60.96 0)
+    (property "Footprint" "Resistor_SMD:R_0603_1608Metric" (at 53.34 60.96 0)
       (effects (font (size 1.27 1.27)) hide)
     )
@@
       (effects (font (size 1.27 1.27)) (justify left))
     )
-    (property "Footprint" "Resistor_SMD:R_0402_1005Metric" (at 88.9 60.96 0)
+    (property "Footprint" "Resistor_SMD:R_0603_1608Metric" (at 88.9 60.96 0)
       (effects (font (size 1.27 1.27)) hide)
     )
@@
       (effects (font (size 1.27 1.27)) (justify left))
     )
-    (property "Footprint" "Resistor_SMD:R_2512_6332Metric" (at 77.47 60.96 0)
+    (property "Footprint" "Resistor_SMD:R_0805_2012Metric" (at 77.47 60.96 0)
       (effects (font (size 1.27 1.27)) hide)
     )
@@
       (effects (font (size 1.27 1.27)) (justify left))
     )
-    (property "Footprint" "Resistor_SMD:R_1210_3225Metric" (at 212.09 109.22 0)
+    (property "Footprint" "Resistor_SMD:R_0603_1608Metric" (at 212.09 109.22 0)
       (effects (font (size 1.27 1.27)) hide)
     )
@@
       (effects (font (size 1.27 1.27)) (justify left))
     )
-    (property "Footprint" "Resistor_SMD:R_1210_3225Metric" (at 207.01 109.22 0)
-      (effects (font (size 1.27 1.27)) hide)
-    )
+    (property "Footprint" "Resistor_SMD:R_0603_1608Metric" (at 207.01 109.22 0)
+      (effects (font (size 1.27 1.27)) hide)
+    )

Commit message: layout update
Parts:
- removed D1: LED, LED_SMD:LED_0805_2012Metric_Pad1.15x1.40mm_HandSolder, symbol PUTRocketLab_semiconductors:LED
- removed R19: 2k, Resistor_SMD:R_0603_1608Metric, symbol PutRocketLab_RCL:R_Small
Other:
- moved on the sheet: 1, D26, D27, R16, R17, R18
