File: keypad-kicad-proj/keypad/io.kicad_sch (KiCad schematic)
At the start: 18 parts, among them SW1 RotaryEncoder, SW2 RotaryEncoder, SW25 SW_RST

Commit message: update datasheets
Parts:
- RV1: value R_Potentiometer_Small -> PTA3043-2010CIB102
Changed lines of the file:
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@@
       (effects (font (size 1.27 1.27)) (justify right))
     )
-    (property "Value" "R_Potentiometer_Small" (at 215.9 46.99 0)
+    (property "Value" "PTA3043-2010CIB102" (at 215.9 46.99 0)
       (effects (font (size 1.27 1.27)) (justify right))
     )
@@
       (effects (font (size 1.27 1.27)) hide)
     )
-    (property "Datasheet" "~" (at 218.44 45.72 0)
+    (property "Datasheet" "https://www.mouser.pl/datasheet/2/54/pta-778345.pdf" (at 218.44 45.72 0)
       (effects (font (size 1.27 1.27)) hide)
     )
