File: keypad-kicad-proj/keypad/keypad.kicad_pcb (KiCad board)
At the start: 2 copper layers, 160 x 125 mm, 103 parts, among them J1 Screw_Terminal_01x02, J2 USB4105-GF-A, J3 USB4105-GF-A, J4 Micro_SD_Card_Det_Hirose_DM3AT, Q1 BC817, Q2 BC817, Q3 IRF9393TRPBF, SW1 RotaryEncoder, SW2 RotaryEncoder, SW25 SW_RST, SW26 Cherry_MX, SW27 Cherry_MX, SW28 Cherry_MX, SW32 Cherry_MX, SW33 Cherry_MX, SW34 Cherry_MX, SW38 Cherry_MX, SW39 Cherry_MX, SW40 Cherry_MX, SW44 Cherry_MX, SW45 Cherry_MX, SW46 Cherry_MX, U1 ESP32-S3-WROOM-1, U10 SK6812MINI-E, U11 SK6812MINI-E, U12 SK6812MINI-E, U13 SK6812MINI-E, U14 SK6812MINI-E, U2 TLV75901PDRVT, U27 SK6812MINI-E, U3 CP2102N-A01-GQFN24, U4 SK6812MINI-E, U5 SK6812MINI-E, U6 SK6812MINI-E, U7 SK6812MINI-E, U8 SK6812MINI-E, U9 SK6812MINI-E

Commit message: update layout
Routing:
- net Net-(Q1-E): track 21.0 -> 72.6 mm, vias 2 -> 4
- net GND: track 0.00 -> 6.53 mm, vias 0 -> 1
- net Net-(D39-A): track 0.00 -> 3.87 mm
- net +3V3: track 280.5 -> 282.0 mm, vias 9 -> 10
- net USB-C_UART_D+: track 48.5 -> 49.6 mm

Commit message: finish routing
Parts:
- moved D25 21.0 mm to (65.3, 62.4)
- moved D24 20.8 mm to (65.3, 60.2)
- moved D23 20.6 mm to (65.3, 58.0)
- moved C6 0.44 mm to (77.0, 53.4)
Routing:
- net GND: track 6.53 -> 9.52 mm, vias 1 -> 28
- net +3V3: track 282.0 -> 284.9 mm
- net Net-(U3-~{RSTb}): track 4.66 -> 6.97 mm
- net USB-C_UART_VBUS: track 140.0 -> 138.6 mm
- net Net-(U3-VBUS): track 10.7 -> 12.0 mm
- net USB-C_UART_D+: track 49.6 -> 48.5 mm
