File: keypad-kicad-proj/keypad/button-matrix.kicad_sch (KiCad schematic)
At the start: 24 parts, among them SW26 Cherry_MX, SW27 Cherry_MX, SW28 Cherry_MX, SW32 Cherry_MX, SW33 Cherry_MX, SW34 Cherry_MX, SW38 Cherry_MX, SW39 Cherry_MX, SW40 Cherry_MX, SW44 Cherry_MX, SW45 Cherry_MX, SW46 Cherry_MX

Commit message: update datasheets
Other:
- note added: "Switches - best if transparent for LED light pass through (e.g. LED Cherry MX) Diodes - 12x 1N4148W-13-F"
Changed lines of the file:
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@@
     (stroke (width 0) (type default))
+  )
+  (text "Switches - best if transparent for LED light pass through (e.g. LED Cherry MX)\nDiodes - 12x 1N4148W-13-F"
+    (at 107.95 144.78 0)
+    (effects (font (size 1.5 1.5)) (justify left bottom))
   )
   (text "Button matrix (4x3)" (at 124.46 45.72 0)
@@
       (effects (font (size 1.27 1.27)) hide)
     )
-    (property "Datasheet" "~" (at 140.97 129.54 90)
+    (property "Datasheet" "https://www.diodes.com/assets/Datasheets/BAV16W_1N4148W.pdf" (at 140.97 129.54 90)
       (effects (font (size 1.27 1.27)) hide)
     )
@@
       (effects (font (size 1.27 1.27)) hide)
     )
-    (property "Datasheet" "~" (at 180.34 129.54 90)
+    (property "Datasheet" "https://www.diodes.com/assets/Datasheets/BAV16W_1N4148W.pdf" (at 180.34 129.54 90)
       (effects (font (size 1.27 1.27)) hide)
     )
@@
       (effects (font (size 1.27 1.27)) hide)
     )
-    (property "Datasheet" "~" (at 218.44 129.54 90)
+    (property "Datasheet" "https://www.diodes.com/assets/Datasheets/BAV16W_1N4148W.pdf" (at 218.44 129.54 90)
       (effects (font (size 1.27 1.27)) hide)
     )
@@
       (effects (font (size 1.27 1.27)) hide)
     )
-    (property "Datasheet" "~" (at 140.97 101.6 90)
+    (property "Datasheet" "https://www.diodes.com/assets/Datasheets/BAV16W_1N4148W.pdf" (at 140.97 101.6 90)
       (effects (font (size 1.27 1.27)) hide)
     )
@@
       (effects (font (size 1.27 1.27)) hide)
     )
-    (property "Datasheet" "~" (at 101.6 129.54 90)
+    (property "Datasheet" "https://www.diodes.com/assets/Datasheets/BAV16W_1N4148W.pdf" (at 101.6 129.54 90)
       (effects (font (size 1.27 1.27)) hide)
     )
@@
       (effects (font (size 1.27 1.27)) hide)
     )
-    (property "Datasheet" "~" (at 101.6 72.39 90)
+    (property "Datasheet" "https://www.diodes.com/assets/Datasheets/BAV16W_1N4148W.pdf" (at 101.6 72.39 90)
       (effects (font (size 1.27 1.27)) hide)
     )
@@
       (effects (font (size 1.27 1.27)) hide)
     )
-    (property "Datasheet" "~" (at 180.34 72.39 90)
+    (property "Datasheet" "https://www.diodes.com/assets/Datasheets/BAV16W_1N4148W.pdf" (at 180.34 72.39 90)
       (effects (font (size 1.27 1.27)) hide)
     )
@@
       (effects (font (size 1.27 1.27)) hide)
     )
-    (property "Datasheet" "~" (at 218.44 101.6 90)
+    (property "Datasheet" "https://www.diodes.com/assets/Datasheets/BAV16W_1N4148W.pdf" (at 218.44 101.6 90)
       (effects (font (size 1.27 1.27)) hide)
     )
@@
       (effects (font (size 1.27 1.27)) hide)
     )
-    (property "Datasheet" "~" (at 180.34 101.6 90)
+    (property "Datasheet" "https://www.diodes.com/assets/Datasheets/BAV16W_1N4148W.pdf" (at 180.34 101.6 90)
       (effects (font (size 1.27 1.27)) hide)
     )
@@
       (effects (font (size 1.27 1.27)) hide)
     )
-    (property "Datasheet" "~" (at 140.97 72.39 90)
+    (property "Datasheet" "https://www.diodes.com/assets/Datasheets/BAV16W_1N4148W.pdf" (at 140.97 72.39 90)
       (effects (font (size 1.27 1.27)) hide)
     )
@@
       (effects (font (size 1.27 1.27)) hide)
     )
-    (property "Datasheet" "~" (at 218.44 72.39 90)
+    (property "Datasheet" "https://www.diodes.com/assets/Datasheets/BAV16W_1N4148W.pdf" (at 218.44 72.39 90)
       (effects (font (size 1.27 1.27)) hide)
     )
@@
       (effects (font (size 1.27 1.27)) hide)
     )
-    (property "Datasheet" "~" (at 101.6 101.6 90)
-      (effects (font (size 1.27 1.27)) hide)
-    )
+    (property "Datasheet" "https://www.diodes.com/assets/Datasheets/BAV16W_1N4148W.pdf" (at 101.6 101.6 90)
+      (effects (font (size 1.27 1.27)) hide)
+    )
