File: kicad-project/keypad/button-matrix.kicad_sch (KiCad schematic)
At the start: 24 parts, among them SW26 Cherry_MX, SW27 Cherry_MX, SW28 Cherry_MX, SW32 Cherry_MX, SW33 Cherry_MX, SW34 Cherry_MX, SW38 Cherry_MX, SW39 Cherry_MX, SW40 Cherry_MX, SW44 Cherry_MX, SW45 Cherry_MX, SW46 Cherry_MX

Commit message: correct schematic
Parts:
- D28, D29, D30, D31, D32, D33, D34, D35, D36, D37, D38, D39: footprint Diode_SMD:D_SOD-123 -> Diode_SMD:D_SOD-323_HandSoldering
Changed lines of the file:
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@@
       (effects (font (size 1.27 1.27)))
     )
-    (property "Footprint" "Diode_SMD:D_SOD-123" (at 140.97 129.54 90)
+    (property "Footprint" "Diode_SMD:D_SOD-323_HandSoldering" (at 140.97 129.54 90)
       (effects (font (size 1.27 1.27)) hide)
     )
@@
       (effects (font (size 1.27 1.27)))
     )
-    (property "Footprint" "Diode_SMD:D_SOD-123" (at 180.34 129.54 90)
+    (property "Footprint" "Diode_SMD:D_SOD-323_HandSoldering" (at 180.34 129.54 90)
       (effects (font (size 1.27 1.27)) hide)
     )
@@
       (effects (font (size 1.27 1.27)))
     )
-    (property "Footprint" "Diode_SMD:D_SOD-123" (at 218.44 129.54 90)
+    (property "Footprint" "Diode_SMD:D_SOD-323_HandSoldering" (at 218.44 129.54 90)
       (effects (font (size 1.27 1.27)) hide)
     )
@@
       (effects (font (size 1.27 1.27)))
     )
-    (property "Footprint" "Diode_SMD:D_SOD-123" (at 140.97 101.6 90)
+    (property "Footprint" "Diode_SMD:D_SOD-323_HandSoldering" (at 140.97 101.6 90)
       (effects (font (size 1.27 1.27)) hide)
     )
@@
       (effects (font (size 1.27 1.27)))
     )
-    (property "Footprint" "Diode_SMD:D_SOD-123" (at 101.6 129.54 90)
+    (property "Footprint" "Diode_SMD:D_SOD-323_HandSoldering" (at 101.6 129.54 90)
       (effects (font (size 1.27 1.27)) hide)
     )
@@
       (effects (font (size 1.27 1.27)))
     )
-    (property "Footprint" "Diode_SMD:D_SOD-123" (at 101.6 72.39 90)
+    (property "Footprint" "Diode_SMD:D_SOD-323_HandSoldering" (at 101.6 72.39 90)
       (effects (font (size 1.27 1.27)) hide)
     )
@@
       (effects (font (size 1.27 1.27)))
     )
-    (property "Footprint" "Diode_SMD:D_SOD-123" (at 180.34 72.39 90)
+    (property "Footprint" "Diode_SMD:D_SOD-323_HandSoldering" (at 180.34 72.39 90)
       (effects (font (size 1.27 1.27)) hide)
     )
@@
       (effects (font (size 1.27 1.27)))
     )
-    (property "Footprint" "Diode_SMD:D_SOD-123" (at 218.44 101.6 90)
+    (property "Footprint" "Diode_SMD:D_SOD-323_HandSoldering" (at 218.44 101.6 90)
       (effects (font (size 1.27 1.27)) hide)
     )
@@
       (effects (font (size 1.27 1.27)))
     )
-    (property "Footprint" "Diode_SMD:D_SOD-123" (at 180.34 101.6 90)
+    (property "Footprint" "Diode_SMD:D_SOD-323_HandSoldering" (at 180.34 101.6 90)
       (effects (font (size 1.27 1.27)) hide)
     )
@@
       (effects (font (size 1.27 1.27)))
     )
-    (property "Footprint" "Diode_SMD:D_SOD-123" (at 140.97 72.39 90)
+    (property "Footprint" "Diode_SMD:D_SOD-323_HandSoldering" (at 140.97 72.39 90)
       (effects (font (size 1.27 1.27)) hide)
     )
@@
       (effects (font (size 1.27 1.27)))
     )
-    (property "Footprint" "Diode_SMD:D_SOD-123" (at 218.44 72.39 90)
+    (property "Footprint" "Diode_SMD:D_SOD-323_HandSoldering" (at 218.44 72.39 90)
       (effects (font (size 1.27 1.27)) hide)
     )
@@
       (effects (font (size 1.27 1.27)))
     )
-    (property "Footprint" "Diode_SMD:D_SOD-123" (at 101.6 101.6 90)
-      (effects (font (size 1.27 1.27)) hide)
-    )
+    (property "Footprint" "Diode_SMD:D_SOD-323_HandSoldering" (at 101.6 101.6 90)
+      (effects (font (size 1.27 1.27)) hide)
+    )
