File: kicad-project/keypad/keypad.kicad_sch (KiCad schematic)
At the start: 3 parts, among them U1 ESP32-S3-WROOM-1

Commit message: correct schematic
Other:
- note added: "INNY PIN!!!"
Changed lines of the file:
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@@
     (effects (font (size 3 3) (thickness 0.6) bold) (justify left bottom))
+  )
+  (text "INNY PIN!!!" (at 93.98 95.25 0)
+    (effects (font (size 1.27 1.27) (thickness 0.254) bold (color 255 104 52 1)) (justify left bottom))
   )
   (global_label "buzzer" (shape output) (at 160.02 83.82 0) (fields_autoplaced)

Commit message: fix board, update production files
Parts:
- C7, C8: footprint Capacitor_SMD:C_0603_1608Metric -> Capacitor_SMD:C_0603_1608Metric_Pad1.08x0.95mm_HandSolder
Connections:
- net SD_DET: now also U1.30 (IO37); no longer U1.26 (IO45)
- net rotary_encoder_1B: now also U1.15 (IO3); no longer U1.16 (IO46)
Other:
- note removed: "INNY PIN!!!"
Changed lines of the file:
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@@
   (no_connect (at 158.75 88.9))
   (no_connect (at 158.75 78.74))
-  (no_connect (at 158.75 76.2))
-  (no_connect (at 158.75 106.68))
   (no_connect (at 128.27 96.52))
   (no_connect (at 128.27 104.14))
   (no_connect (at 158.75 81.28))
   (no_connect (at 128.27 99.06))
+  (no_connect (at 158.75 106.68))
   (no_connect (at 158.75 109.22))
-  (no_connect (at 128.27 101.6))
+  (no_connect (at 128.27 116.84))
+  (no_connect (at 128.27 93.98))
   (wire (pts (xy 140.97 127) (xy 140.97 130.81))
     (stroke (width 0) (type default))
@@
     (stroke (width 0) (type default))
   )
-  (wire (pts (xy 127 116.84) (xy 128.27 116.84))
-    (stroke (width 0) (type default))
-  )
   (wire (pts (xy 143.51 54.61) (xy 147.32 54.61))
     (stroke (width 0) (type default))
@@
   )
   (wire (pts (xy 127 121.92) (xy 128.27 121.92))
-    (stroke (width 0) (type default))
-  )
-  (wire (pts (xy 127 93.98) (xy 128.27 93.98))
     (stroke (width 0) (type default))
   )
@@
     (effects (font (size 3 3) (thickness 0.6) bold) (justify left bottom))
   )
-  (text "INNY PIN!!!" (at 93.98 95.25 0)
-    (effects (font (size 1.27 1.27) (thickness 0.254) bold (color 255 104 52 1)) (justify left bottom))
-  )
   (global_label "buzzer" (shape output) (at 160.02 83.82 0) (fields_autoplaced)
     (effects (font (size 1.27 1.27)) (justify left))
@@
     )
   )
-  (global_label "rotary_encoder_1B" (shape bidirectional) (at 127 93.98 180) (fields_autoplaced)
-    (effects (font (size 1.27 1.27)) (justify right))
-    (property "Intersheetrefs" "${INTERSHEET_REFS}" (at 105.4261 93.98 0)
-      (effects (font (size 1.27 1.27)) (justify right) hide)
-    )
-  )
-  (global_label "SD_DET" (shape input) (at 127 116.84 180) (fields_autoplaced)
-    (effects (font (size 1.27 1.27)) (justify right))
-    (property "Intersheetrefs" "${INTERSHEET_REFS}" (at 117.1811 116.84 0)
+  (global_label "rotary_encoder_1B" (shape bidirectional) (at 158.75 76.2 0) (fields_autoplaced)
+    (effects (font (size 1.27 1.27)) (justify left))
+    (property "Intersheetrefs" "${INTERSHEET_REFS}" (at 180.3239 76.2 0)
+      (effects (font (size 1.27 1.27)) (justify left) hide)
+    )
+  )
+  (global_label "SD_DET" (shape input) (at 128.27 101.6 180) (fields_autoplaced)
+    (effects (font (size 1.27 1.27)) (justify right))
+    (property "Intersheetrefs" "${INTERSHEET_REFS}" (at 118.4511 101.6 0)
       (effects (font (size 1.27 1.27)) (justify right) hide)
     )
@@
       (effects (font (size 1.27 1.27)) (justify left))
     )
-    (property "Footprint" "Capacitor_SMD:C_0603_1608Metric" (at 147.32 58.42 0)
+    (property "Footprint" "Capacitor_SMD:C_0603_1608Metric_Pad1.08x0.95mm_HandSolder" (at 147.32 58.42 0)
       (effects (font (size 1.27 1.27)) hide)
     )
@@
       (effects (font (size 1.27 1.27)) (justify left))
     )
-    (property "Footprint" "Capacitor_SMD:C_0603_1608Metric" (at 139.7 58.42 0)
-      (effects (font (size 1.27 1.27)) hide)
-    )
+    (property "Footprint" "Capacitor_SMD:C_0603_1608Metric_Pad1.08x0.95mm_HandSolder" (at 139.7 58.42 0)
+      (effects (font (size 1.27 1.27)) hide)
+    )
