File: kicad-project/keypad/micro-sd-connector.kicad_sch (KiCad schematic)
At the start: 8 parts, among them J4 Micro_SD_Card_Det_Hirose_DM3AT

Commit message: fix board, update production files
Parts:
- C10: footprint Capacitor_SMD:C_0603_1608Metric -> Capacitor_SMD:C_0603_1608Metric_Pad1.08x0.95mm_HandSolder
Changed lines of the file:
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@@
       (effects (font (size 1.27 1.27)) (justify left))
     )
-    (property "Footprint" "Capacitor_SMD:C_0603_1608Metric" (at 135.89 100.33 0)
+    (property "Footprint" "Capacitor_SMD:C_0603_1608Metric_Pad1.08x0.95mm_HandSolder" (at 135.89 100.33 0)
       (effects (font (size 1.27 1.27)) hide)
     )
