File: kicad-project/keypad/usb-c-interface.kicad_sch (KiCad schematic)
At the start: 25 parts, among them J2 USB4105-GF-A, Q1 BC817, Q2 BC817, U3 CP2102N-A01-GQFN24

Commit message: update project
Other:
- moved on the sheet: C4, D18, D20

Commit message: correct schematic
Parts:
- added C20: 1uF, Capacitor_SMD:C_0603_1608Metric, symbol PutRocketLab_RCL:C_Small
- added R25: 10k, Resistor_SMD:R_0603_1608Metric, symbol PutRocketLab_RCL:R_Small
- added R26, R27: 5.1k, Capacitor_SMD:C_0805_2012Metric, symbol PutRocketLab_RCL:R_Small
- R22, R23: value 56k -> 5.1k
Connections:
- net +3V3: now also R25.2
- net GND: now also R22.2, R23.2, C20.2, R26.2, R27.2
- net RTS: now also C20.1, R25.1
- net USB-C_UART_VBUS: no longer R22.1
- net at Q1.2 (E), R11.2: now also U3.19 (RTS); no longer U3.23 (DTR)
- net at D17.2 (A), J2.A4_B9 (VBUS), J2.B4_A9 (VBUS): no longer R23.1
- net at Q2.2 (E), R10.2: now also U3.23 (DTR); no longer U3.19 (RTS)
- new net: J2.A5 (CC1), R22.1
- new net: J2.B5 (CC2), R27.1
- new net: J2.A5 (CC1), R23.1
- new net: J2.B5 (CC2), R26.1
Other:
- moved on the sheet: C3, C5, C6, D14, D15, D16, D17, J2, Q1, Q2, R10, R11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

Commit message: fix board, update production files
Parts:
- C20, C3, C4, C5, C6: footprint Capacitor_SMD:C_0603_1608Metric -> Capacitor_SMD:C_0603_1608Metric_Pad1.08x0.95mm_HandSolder
Changed lines of the file:
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@@
       (effects (font (size 1.27 1.27)) (justify left))
     )
-    (property "Footprint" "Capacitor_SMD:C_0603_1608Metric" (at 142.24 43.18 0)
+    (property "Footprint" "Capacitor_SMD:C_0603_1608Metric_Pad1.08x0.95mm_HandSolder" (at 142.24 43.18 0)
       (effects (font (size 1.27 1.27)) hide)
     )
@@
       (effects (font (size 1.27 1.27)) (justify left))
     )
-    (property "Footprint" "Capacitor_SMD:C_0603_1608Metric" (at 148.59 111.76 0)
+    (property "Footprint" "Capacitor_SMD:C_0603_1608Metric_Pad1.08x0.95mm_HandSolder" (at 148.59 111.76 0)
       (effects (font (size 1.27 1.27)) hide)
     )
@@
       (effects (font (size 1.27 1.27)) (justify left))
     )
-    (property "Footprint" "Capacitor_SMD:C_0603_1608Metric" (at 144.78 146.05 0)
+    (property "Footprint" "Capacitor_SMD:C_0603_1608Metric_Pad1.08x0.95mm_HandSolder" (at 144.78 146.05 0)
       (effects (font (size 1.27 1.27)) hide)
     )
@@
       (effects (font (size 1.27 1.27)))
     )
-    (property "Footprint" "Capacitor_SMD:C_0603_1608Metric" (at 252.73 86.36 0)
+    (property "Footprint" "Capacitor_SMD:C_0603_1608Metric_Pad1.08x0.95mm_HandSolder" (at 252.73 86.36 0)
       (effects (font (size 1.27 1.27)) hide)
     )
@@
       (effects (font (size 1.27 1.27)))
     )
-    (property "Footprint" "Capacitor_SMD:C_0603_1608Metric" (at 170.18 74.93 0)
-      (effects (font (size 1.27 1.27)) hide)
-    )
+    (property "Footprint" "Capacitor_SMD:C_0603_1608Metric_Pad1.08x0.95mm_HandSolder" (at 170.18 74.93 0)
+      (effects (font (size 1.27 1.27)) hide)
+    )
